File: Hardware/_autosave-sm4.kicad_pcb (KiCad board)
At the start: 4 copper layers, 50 x 45 mm, 94 parts, among them J1 Motor1, J2 Termination, J3 CAN bus, J4 Motor2, J5 I2C, J6 Power, J7 USB_C_Receptacle_USB2.0, Q1 NDT2955, SW1 RST_SW, SW2 BOOT_SW, U1 STM32F412RETx, U2 TMC2100-TA, U3 MCP2562-E-SN, U4 TMC2100-TA, U5 LM2594HVM-5.0, U6 MCP1700-3302E_SOT23, U7 USBLC6-2SC6, Y1 25 MHz

Commit message: Finish first version of the PCB, which is trash and shall perish.
Parts:
- removed C33: 100u, Capacitor_SMD:C_Elec_6.3x5.8
- removed D2: B0520LW, Diode_SMD:D_SOD-123
- removed L1: 100uH, Inductor_SMD:L_Wuerth_HCI-1050
- removed U5: LM2594HVM-5.0, Package_SO:SOIC-8_3.9x4.9mm_P1.27mm
- added J8: Conn_01x05_Male, Connector_Molex:Molex_SPOX_5267-05A_1x05_P2.50mm_Vertical, F.Cu at (131.8, 78.2)
- C10, C30, C32, C7: footprint Capacitor_SMD:C_0805_2012Metric_Pad1.18x1.45mm_HandSolder -> Capacitor_SMD:C_0603_1608Metric_Pad1.08x0.95mm_HandSolder; moved to B.Cu
- C11, C18, C2, C23, C24, C25, C26, C27, C28, C29, C3, C31, C34, C35, C4, C5, C6, C8, C9, D1, D3, FB2, J7, R1, R14, R15, R16, R17, R2, R22, R3, R4, R5, R9: moved to B.Cu
- F1: footprint Fuse:Fuse_2920_7451Metric_Pad2.10x5.45mm_HandSolder -> Fuse:Fuse_1206_3216Metric_Pad1.42x1.75mm_HandSolder; moved to B.Cu
- SW1: footprint Button_Switch_SMD:SW_Push_1P1T_NO_6x6mm_H9.5mm -> Connector_PinHeader_2.54mm:PinHeader_1x02_P2.54mm_Vertical
- moved C4 113.9 mm to (125.5, 88.2), turned to 180 degrees
- moved R23 106.3 mm to (122.6, 62.1)
- moved U6 103.0 mm to (131.5, 53.5), turned to 270 degrees
- moved Q1 102.4 mm to (175.4, 53.4)
- moved F2 99.4 mm to (129.8, 60.1), turned to 180 degrees
- moved D4 99.3 mm to (129.7, 57.4), turned to 180 degrees
- moved R22 98.9 mm to (128.0, 66.7), turned to 90 degrees
- moved C8 96.5 mm to (135.6, 68.3), turned to 270 degrees
- moved C1 95.0 mm to (139.0, 53.4), turned to 90 degrees
- moved C12 93.8 mm to (137.2, 53.4), turned to 90 degrees
- moved R4 91.4 mm to (143.4, 64.9), turned to 270 degrees
- moved C34 91.3 mm to (128.6, 53.5), turned to 90 degrees
- moved C13 90.2 mm to (151.6, 59.2), turned to 90 degrees
- moved C9 89.5 mm to (136.2, 88.3), turned to 270 degrees
- moved R6 88.5 mm to (150.8, 62.0)
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Connections:
- D3 pad 2: Net-(C33-Pad1) -> Net-(C25-Pad1)
- J3 pad 4: +5V -> VDC
- J5 pad 2: (no net) -> SCL
- J5 pad 3: (no net) -> SDA
- J5 pad 4: +5V -> VDC
- Q1 pad 3: VS1 -> VDC
- R21 pad 2: (no net) -> STATUS
- R24 pad 2: (no net) -> ERR
- U1 pad 10: (no net) -> CFG02
- U1 pad 11: (no net) -> DIR2
- U1 pad 14: (no net) -> VBAT
- U1 pad 15: (no net) -> CFG52
- U1 pad 16: (no net) -> CFG42
- U1 pad 17: (no net) -> ERR2
- U1 pad 2: (no net) -> STATUS
- U1 pad 3: (no net) -> ERR
- U1 pad 4: (no net) -> CFG32
- U1 pad 40: (no net) -> SDA
- U1 pad 41: (no net) -> SCL
- U1 pad 42: (no net) -> CFG41
- U1 pad 43: (no net) -> CFG51
- U1 pad 46: (no net) -> SWDIO
- U1 pad 49: (no net) -> SWCLK
- U1 pad 51: (no net) -> CFG31
- U1 pad 52: (no net) -> CFG21
- U1 pad 53: (no net) -> CFG11
- U1 pad 55: (no net) -> CFG01
- U1 pad 56: (no net) -> STEP1
- U1 pad 57: (no net) -> DIR1
- U1 pad 58: (no net) -> STEP2
- U1 pad 59: (no net) -> ERR1
- U1 pad 61: (no net) -> CAN_RX
- U1 pad 62: (no net) -> CAN_TX
- U1 pad 8: (no net) -> CFG22
- U1 pad 9: (no net) -> CFG12
- U2 pad 24: (no net) -> CFG41
- U2 pad 25: (no net) -> CFG51
- U2 pad 3: (no net) -> CFG31
- U2 pad 4: (no net) -> CFG21
- U2 pad 5: (no net) -> CFG11
- U2 pad 7: (no net) -> CFG01
- U2 pad 8: (no net) -> STEP1
- U2 pad 9: (no net) -> DIR1
- U3 pad 1: (no net) -> CAN_TX
- U3 pad 4: (no net) -> CAN_RX
- U4 pad 24: (no net) -> CFG42
- U4 pad 25: (no net) -> CFG52
- U4 pad 3: (no net) -> CFG32
- U4 pad 4: (no net) -> CFG22
- U4 pad 5: (no net) -> CFG12
- U4 pad 7: (no net) -> CFG02
- U4 pad 8: (no net) -> STEP2
- U4 pad 9: (no net) -> DIR2
- U6 pad 1: (no net) -> GND
Routing:
- net VS1: track 0.00 -> 111.1 mm, vias 0 -> 6
- net GND: track 0.00 -> 110.9 mm, vias 0 -> 78
- net ERR2: track 0.00 -> 59.0 mm, vias 0 -> 3
- net SCL: track 0.00 -> 58.5 mm, vias 0 -> 1
- net SDA: track 0.00 -> 57.4 mm, vias 0 -> 1
- net +5V: track 0.00 -> 56.3 mm, vias 0 -> 3
- net NRST: track 0.00 -> 47.1 mm, vias 0 -> 1
- net VBAT: track 0.00 -> 43.9 mm, vias 0 -> 4
- net CFG42: track 0.00 -> 43.5 mm, vias 0 -> 3
- net CFG52: track 0.00 -> 37.9 mm, vias 0 -> 3
- net DIR2: track 0.00 -> 35.8 mm, vias 0 -> 1
- net CFG02: track 0.00 -> 35.5 mm, vias 0 -> 3
- net CFG12: track 0.00 -> 33.5 mm, vias 0 -> 3
- net CFG22: track 0.00 -> 31.9 mm, vias 0 -> 3
- net Net-(J1-Pad4): track 0.00 -> 31.8 mm
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Other:
- board size 50 x 45 mm -> 65 x 50 mm
