File: Hardware/sm4.sch (KiCad schematic (older format))
At the start: 5 parts

Commit message: Start working on the schematic.
Parts:
- added C1: 2u2, symbol Device:C_Small
- added C10, C11, C12, C4, C7: 100n, symbol Device:C_Small
- added C13, C16, C17, C5: 1u, symbol Device:C_Small
- added C14, C15: 68u, symbol Device:C_Small
- added C2: 4u7, symbol Device:C_Small
- added C3, C8: 10n, symbol Device:C_Small
- added C6, C9: 22p, symbol Device:C_Small
- added D1: 4V7, symbol Device:D_Zener_Small
- added D2: 1N5817, Diode_THT:D_DO-41_SOD81_P10.16mm_Horizontal, symbol Diode:1N5817
- added D3, D4: D_Small, symbol Device:D_Small
- added F1: 500mA, symbol Device:Polyfuse_Small
- added FB1, FB2: 1k @ 100 MHz, symbol Device:Ferrite_Bead_Small
- added H1, H2, H3, H4: MountingHole_Pad, symbol Mechanical:MountingHole_Pad
- added L1: 100uH, symbol Device:L_Small
- added Q1: NDT2955, Package_TO_SOT_SMD:SOT-23, symbol Transistor_FET:AO3401A
- added R1, R3: 10k, symbol Device:R_Small
- added R2: 47R, symbol Device:R_Small
- added SW1: RST_SW, symbol Switch:SW_SPST
- added SW2: BOOT_SW, symbol Switch:SW_SPDT
- added Y1: 25 MHz, symbol Device:Crystal_GND24_Small
- gave numbers to parts that had none: 5
Connections:
- net +3V3: now reaches U1.1 (VBAT)
- net +3V3: now also U1.19 (VDD), U1.32 (VDD), U1.48 (VDD), U1.64 (VDD), U5.2 (VO), C10.1, C11.1, C12.1, C17.1, C2.1, C4.1, C7.1, FB1.2, SW2.1 (A)
- net GND: now reaches U1.12 (VSSA)
- net GND: now also U1.18 (VSS), U1.31 (VSS), U1.47 (VSS), U1.63 (VSS), U4.5 (~ON~/OFF), U4.6 (GND), C1.2, C10.2, C11.2, C12.2, C13.2, C14.2, C15.2, C16.2, C17.2, C2.2, C3.2, C4.2, C5.2, C6.2, C7.2, C8.2, C9.2, D2.2 (A), H1.1, H2.1, H3.1, H4.1, R3.1, SW1.2 (B), SW2.3 (C), Y1.2, Y1.4
- net VDDA: now reaches U1.13 (VDDA)
- net VDDA: now also C5.1, C8.1, FB1.1
- net at U1.30 (VCAP_1): now also C1.1
- net USB_D-: now reaches U1.44 (PA11)
- net USB_D+: now reaches U1.45 (PA12)
- net OSC_IN: now reaches U1.5 (PH0)
- net OSC_IN: now also C6.1, Y1.1
- net OSC_OUT: now reaches U1.6 (PH1)
- net OSC_OUT: now also R2.1
- net BOOT: now reaches U1.60 (BOOT0)
- net BOOT: now also R1.2
- net NRST: now reaches U1.7 (NRST)
- net NRST: now also C3.1, SW1.1 (A)
- net at U4.7 (VIN): now also C13.1, C14.1, FB2.1
- net at U4.8 (OUT): now also D2.1 (K), L1.1
- net +5V: now reaches U5.3 (VI)
- net +5V: now also C16.1, D3.1 (K), D4.1 (K)
- new net: R1.1, SW2.2 (B)
- new net: C9.1, R2.2, Y1.3
- new net: D1.2 (A), Q1.1 (G), R3.2
- new net: D1.1 (K), F1.2, Q1.2 (S)
- new net: F1.1, FB2.2
- new net: C15.1, D3.2 (A), L1.2
- new net +5VD: D4.2 (A)
- new net VCC: Q1.3 (D)
Other:
- note added: "Controller and its connections"
- note added: "Controller power filtering"
- note added: "DLG-0504-101"
- note added: "Determine values for oscillator!"
- note added: "Hodnoty pro ferity"
- note added: "Mounting"
- note added: "Power source"
- note added: "Supplementary controller circuitry"
- note added: "TODO"
- note added: "vybrat shottky\n"
- moved on the sheet: U1, U2, U3, U4, U5

Commit message: Add circuitry for the motor controllers.
Parts:
- removed U3: TMC2100-TA, Package_QFP:TQFP-48-1EP_7x7mm_P0.5mm_EP5x5mm_ThermalVias, symbol Driver_Motor:TMC2100-TA
- added C10, C7, C? (x2): 470n, symbol Device:C_Small
- added C2, C3, C5, C6, C? (x4): 100n, symbol Device:C_Small
- added C4, C?: 100u, symbol Device:C_Small
- added C9, C?: 22n@50V, symbol Device:C_Small
- added J1: Motor1, symbol Connector:Conn_01x04_Male
- added J?: Motor2, symbol Connector:Conn_01x04_Male
- added R1, R?: 10k, symbol Device:R_Small
- added R2, R?: 2R2, symbol Device:R_Small
- added R3, R5, R? (x2): 1R, symbol Device:R_Small
- added U?: TMC2100-TA, Package_QFP:TQFP-48-1EP_7x7mm_P0.5mm_EP5x5mm_ThermalVias, symbol Driver_Motor:TMC2100-TA
- renumbered C3 to C11, C4 to C12, C5 to C13, C6 to C14, C7 to C15, C8 to C16, C9 to C17, C10 to C18, C11 to C19, C12 to C20, C13 to C21, C14 to C22, C15 to C23, C16 to C24, C17 to C25, C2 to C8, R1 to R4, R2 to R6, R3 to R7, U4 to U3, U5 to U4
Connections:
- net +3V3: now also U2.10 (VCC_IO), R1.2, R?.2, U?.10 (VCC_IO)
- net GND: now also U2.1 (TST_MODE), U2.12 (GNDD), U2.13 (GNDP), U2.2 (CLK), U2.31 (GNDD), U2.32 (GNDA), U2.36 (GNDD), U2.48 (GNDP), U2.49 (GNDD), U2.6 (GNDD), C10.2, C4.2, C5.2, C6.2, C7.2, C?.2, C?.2, C?.2, C?.2, C?.2, R3.1, R5.1, R?.1, R?.1, U?.1 (TST_MODE), U?.12 (GNDD), U?.13 (GNDP), U?.2 (CLK), U?.31 (GNDD), U?.32 (GNDA), U?.36 (GNDD), U?.48 (GNDP), U?.49 (GNDD), U?.6 (GNDD)
- net VCC: now also U2.21 (VS), U2.40 (VS), C2.1, C3.1, C4.1, C5.1, C6.1, C?.1, C?.1, C?.1, C?.1, C?.1, U?.21 (VS), U?.40 (VS)
- net at U2.15 (OB1): now also J1.1 (Pin_1)
- net at U2.17 (BRB): now also R3.2
- net at U2.19 (OB2): now also J1.2 (Pin_2)
- net CFG41: now reaches U2.24 (CFG4)
- net CFG51: now reaches U2.25 (CFG5)
- net ERR1: now reaches U2.26 (ERROR)
- net ERR1: now also R1.1
- net CFG61: now reaches U2.29 (~CFG6_ENN)
- net CFG31: now reaches U2.3 (CFG3)
- net VREF1: now reaches U2.30 (AIN_REF)
- net 5VOUT1: now reaches U2.33 (5VOUT)
- net 5VOUT1: now also C7.1, R2.1
- net 5VM1: now reaches U2.34 (VCC)
- net 5VM1: now also C10.1, R2.2
- net at U2.35 (CP0): now also C9.2
- net at U2.37 (CPI): now also C9.1
- net VCP1: now reaches U2.38 (VCP)
- net VCP1: now also C2.2
- net VSA1: now reaches U2.39 (VSA)
- net VSA1: now also C3.2
- net at U2.42 (OA2): now also J1.3 (Pin_3)
- net at U2.44 (BRA): now also R5.2
- net at U2.46 (OA1): now also J1.4 (Pin_4)
- net CFG11: now reaches U2.5 (CFG1)
- net CFG01: now reaches U2.7 (CFG0)
- net STEP1: now reaches U2.8 (STEP)
- net DIR1: now reaches U2.9 (DIR)
- new net: J?.1 (Pin_1), U?.15 (OB1)
- new net: J?.2 (Pin_2), U?.19 (OB2)
- new net: J?.3 (Pin_3), U?.42 (OA2)
- new net: J?.4 (Pin_4), U?.46 (OA1)
- new net: C?.1, U?.37 (CPI)
- new net: C?.2, U?.35 (CP0)
- new net: R?.2, U?.17 (BRB)
- new net: R?.2, U?.44 (BRA)
- new net 5VM2: C?.1, R?.2, U?.34 (VCC)
- new net 5VOUT2: C?.1, R?.1, U?.33 (5VOUT)
- new net CFG02: U?.7 (CFG0)
- new net CFG12: U?.5 (CFG1)
- new net CFG32: U?.3 (CFG3)
- new net CFG42: U?.24 (CFG4)
- new net CFG52: U?.25 (CFG5)
- new net CFG62: U?.29 (~CFG6_ENN)
- new net DIR2: U?.9 (DIR)
- new net ERR2: R?.1, U?.26 (ERROR)
- new net STEP2: U?.8 (STEP)
- new net VCP2: C?.2, U?.38 (VCP)
- new net VREF2: U?.30 (AIN_REF)
- new net VSA2: C?.2, U?.39 (VSA)
- no-connect marks 0 -> 4
Other:
- note added: "CAN bus"
- note added: "Motor controller 1"
- note added: "Motor controller 2"
- note added: "Reverse V protection for motor drivers"
- note added: "snimani napeti baterie"
- moved on the sheet: U2

Commit message: Add packages to components.
Parts:
- added C21, C22: 100n, Capacitor_SMD:C_0603_1608Metric_Pad1.08x0.95mm_HandSolder, symbol Device:C_Small
- added C36: 10n, Capacitor_SMD:C_0603_1608Metric_Pad1.08x0.95mm_HandSolder, symbol Device:C_Small
- added D5, D6, D7: LED_Small, LED_SMD:LED_0603_1608Metric_Pad1.05x0.95mm_HandSolder, symbol Device:LED_Small
- added F2: 500mA, Fuse:Fuse_1206_3216Metric_Pad1.42x1.75mm_HandSolder, symbol Device:Polyfuse_Small
- added J2: Termination, Connector_PinHeader_2.54mm:PinHeader_1x02_P2.54mm_Vertical, symbol Connector:Conn_01x02_Male
- added J3: CAN bus, Connector_Molex:Molex_SPOX_5268-04A_1x04_P2.50mm_Horizontal, symbol Connector:Conn_01x04_Male
- added J5: I2C, Connector_Molex:Molex_SPOX_5268-04A_1x04_P2.50mm_Horizontal, symbol Connector:Conn_01x04_Male
- added J6: Power, TerminalBlock:TerminalBlock_bornier-2_P5.08mm, symbol Connector:Screw_Terminal_01x02
- added J7: USB_C_Receptacle_USB2.0, Connector_USB:USB_C_Receptacle_GCT_USB4085, symbol Connector:USB_C_Receptacle_USB2.0
- added R10, R8: 1M, Resistor_SMD:R_0603_1608Metric_Pad0.98x0.95mm_HandSolder, symbol Device:R_Small
- added R11, R7: 0R, Resistor_SMD:R_0603_1608Metric_Pad0.98x0.95mm_HandSolder, symbol Device:R_Small
- added R12, R13: 47R9, Resistor_SMD:R_0603_1608Metric_Pad0.98x0.95mm_HandSolder, symbol Device:R_Small
- added R18: 100k, Resistor_SMD:R_0603_1608Metric_Pad0.98x0.95mm_HandSolder, symbol Device:R_Small
- added R19: 4k7, Resistor_SMD:R_0603_1608Metric_Pad0.98x0.95mm_HandSolder, symbol Device:R_Small
- added R20, R21, R24: 1k, Resistor_SMD:R_0603_1608Metric_Pad0.98x0.95mm_HandSolder, symbol Device:R_Small
- added R22, R23: 5k1, Resistor_SMD:R_0603_1608Metric_Pad0.98x0.95mm_HandSolder, symbol Device:R_Small
- added U3: MCP2562-E-SN, Package_SO:SOIC-8_3.9x4.9mm_P1.27mm, symbol Interface_CAN_LIN:MCP2562-E-SN
- added U7: USBLC6-2SC6, Package_TO_SOT_SMD:SOT-23-6, symbol Power_Protection:USBLC6-2SC6
- C1, C11, C12, C13, C15, C16, C18, C19, C20, C8, C9: footprint (none) -> Capacitor_SMD:C_0603_1608Metric_Pad1.08x0.95mm_HandSolder
- C10, C2, C3, C5, C6, C7: footprint (none) -> Capacitor_SMD:C_0805_2012Metric_Pad1.18x1.45mm_HandSolder
- C14, C17: value 22p -> 12p; footprint (none) -> Capacitor_SMD:C_0603_1608Metric_Pad1.08x0.95mm_HandSolder
- C23, C24, C28, C29, C30, C32: renamed from C?; footprint (none) -> Capacitor_SMD:C_0805_2012Metric_Pad1.18x1.45mm_HandSolder
- C25: renamed from C21; footprint (none) -> Capacitor_SMD:C_1206_3216Metric_Pad1.33x1.80mm_HandSolder
- C26: renamed from C?; value 100u -> 47u; footprint (none) -> Capacitor_SMD:C_Elec_8x6.2
- C27: renamed from C22; footprint (none) -> Capacitor_SMD:C_Elec_6.3x7.7
- C31: renamed from C?; footprint (none) -> Capacitor_SMD:C_0603_1608Metric_Pad1.08x0.95mm_HandSolder
- C33: renamed from C23; value 68u -> 100u; footprint (none) -> Capacitor_SMD:C_Elec_6.3x5.8
- C34: renamed from C24; footprint (none) -> Capacitor_SMD:C_0603_1608Metric_Pad1.08x0.95mm_HandSolder
- C35: renamed from C25; footprint (none) -> Capacitor_SMD:C_0603_1608Metric_Pad1.08x0.95mm_HandSolder
- C4: value 100u -> 47u; footprint (none) -> Capacitor_SMD:C_Elec_8x6.2
- D1, D3, D4: footprint (none) -> Diode_SMD:D_SOD-123
- D2: value 1N5817 -> B0520LW; footprint Diode_THT:D_DO-41_SOD81_P10.16mm_Horizontal -> Diode_SMD:D_SOD-123
- F1: footprint (none) -> Fuse:Fuse_2920_7451Metric_Pad2.10x5.45mm_HandSolder
- FB1, FB2, R1, R2, R3, R4, R5, R6: footprint (none) -> Resistor_SMD:R_0603_1608Metric_Pad0.98x0.95mm_HandSolder
- H1, H2, H3, H4: footprint (none) -> MountingHole:MountingHole_3.2mm_M3_Pad
- J1: footprint (none) -> Connector_PinHeader_2.54mm:PinHeader_1x04_P2.54mm_Horizontal
- J4: renamed from J?; footprint (none) -> Connector_PinHeader_2.54mm:PinHeader_1x04_P2.54mm_Horizontal
- L1: footprint (none) -> Inductor_SMD:L_Wuerth_HCI-1050
- R14, R15, R16, R17: renamed from R?; footprint (none) -> Resistor_SMD:R_0603_1608Metric_Pad0.98x0.95mm_HandSolder
- R9: renamed from R7; footprint (none) -> Resistor_SMD:R_0603_1608Metric_Pad0.98x0.95mm_HandSolder
- SW1: footprint (none) -> Button_Switch_SMD:SW_Push_1P1T_NO_6x6mm_H9.5mm
- SW2: footprint (none) -> Button_Switch_SMD:SW_SPDT_PCM12
- Y1: footprint (none) -> Crystal:Crystal_SMD_3225-4Pin_3.2x2.5mm_HandSoldering
- gave numbers to parts that had none: 1
- renumbered U3 to U5, U4 to U6
Connections:
- net +3V3: now also C21.1, R10.1, R20.2, R7.1
- net +5V: now also C22.1, J3.4 (Pin_4), J5.4 (Pin_4), U3.3 (VDD)
- net +5VD: now also F2.1, U7.5 (VBUS)
- net GND: now also C21.2, C22.2, C36.2, D5.1 (K), D6.1 (K), D7.1 (K), J3.1 (Pin_1), J5.1 (Pin_1), J6.1 (Pin_1), J7.A1 (GND), J7.A12 (GND), J7.B1 (GND), J7.B12 (GND), J7.S1 (SHIELD), R11.2, R19.1, R22.1, R23.1, R8.2, U3.2 (VSS), U7.2 (GND)
- net USB_D+: now also U7.4 (I/O2)
- net USB_D-: now also U7.6 (I/O1)
- net VCC: now also J6.2 (Pin_2), R18.2
- new net: F2.2, J7.A4 (VBUS), J7.A9 (VBUS), J7.B4 (VBUS), J7.B9 (VBUS)
- new net: J7.A5 (CC1), R22.2
- new net: J7.B5 (CC2), R23.2
- new net: D5.2 (A), R20.1
- new net: D6.2 (A), R21.1
- new net: D7.2 (A), R24.1
- new net: R7.2, R8.1, U3.5 (Vio)
- new net: J3.2 (Pin_2), R13.2, U3.6 (CANL)
- new net: J3.3 (Pin_3), R12.2, U3.7 (CANH)
- new net: R10.2, R11.1, U3.8 (STBY)
- new net: J2.2 (Pin_2), R12.1
- new net: J2.1 (Pin_1), R13.1
- new net CAN_RX: U3.4 (RXD)
- new net CAN_TX: U3.1 (TXD)
- new net ERR: R24.2
- new net SCL: J5.2 (Pin_2)
- new net SDA: J5.3 (Pin_3)
- new net STATUS: R21.2
- new net USB_CONN_D+: J7.A6 (D+), J7.B6 (D+), U7.3 (I/O2)
- new net USB_CONN_D-: J7.A7 (D-), J7.B7 (D-), U7.1 (I/O1)
- new net VBAT: C36.1, R18.1, R19.2
- no-connect marks 4 -> 6
Other:
- note added: "Power terminal"
- note added: "USB"
- note removed: "snimani napeti baterie"

Commit message: Finish first version of the PCB, which is trash and shall perish.
Parts:
- removed C33: 100u, Capacitor_SMD:C_Elec_6.3x5.8, symbol Device:C_Small
- removed D2: B0520LW, Diode_SMD:D_SOD-123, symbol Diode:1N5817
- removed L1: 100uH, Inductor_SMD:L_Wuerth_HCI-1050, symbol Device:L_Small
- removed U5: LM2594HVM-5.0, Package_SO:SOIC-8_3.9x4.9mm_P1.27mm, symbol Regulator_Switching:LM2594HVM-5.0
- added J8: Conn_01x05_Male, Connector_Molex:Molex_SPOX_5267-05A_1x05_P2.50mm_Vertical, symbol Connector:Conn_01x05_Male
- C10, C30, C32, C7: footprint Capacitor_SMD:C_0805_2012Metric_Pad1.18x1.45mm_HandSolder -> Capacitor_SMD:C_0603_1608Metric_Pad1.08x0.95mm_HandSolder
- F1: footprint Fuse:Fuse_2920_7451Metric_Pad2.10x5.45mm_HandSolder -> Fuse:Fuse_1206_3216Metric_Pad1.42x1.75mm_HandSolder
- SW1: footprint Button_Switch_SMD:SW_Push_1P1T_NO_6x6mm_H9.5mm -> Connector_PinHeader_2.54mm:PinHeader_1x02_P2.54mm_Vertical
Connections:
- net +3V3: now also J8.5 (Pin_5)
- net +5V: no longer J3.4 (Pin_4), J5.4 (Pin_4)
- net CAN_RX: now also U1.61 (PB8)
- net CAN_TX: now also U1.62 (PB9)
- net CFG01: now also U1.55 (PB3)
- net CFG02: now also U1.10 (PC2)
- net CFG11: now also U1.53 (PC12)
- net CFG12: now also U1.9 (PC1)
- net CFG31: now also U1.51 (PC10)
- net CFG32: now also U1.4 (PC15)
- net CFG41: now also U1.42 (PA9)
- net CFG42: now also U1.16 (PA2)
- net CFG51: now also U1.43 (PA10)
- net CFG52: now also U1.15 (PA1)
- net DIR1: now also U1.57 (PB5)
- net DIR2: now also U1.11 (PC3)
- net ERR: now also U1.3 (PC14)
- net ERR1: now also U1.59 (PB7)
- net ERR2: now also U1.17 (PA3)
- net GND: now also U6.1 (GND), J8.3 (Pin_3)
- net NRST: now also J8.1 (Pin_1)
- net SCL: now also U1.41 (PA8)
- net SDA: now also U1.40 (PC9)
- net STATUS: now also U1.2 (PC13)
- net STEP1: now also U1.56 (PB4)
- net STEP2: now also U1.58 (PB6)
- net VBAT: now also U1.14 (PA0)
- net VCC: no longer Q1.3 (D)
- net SWDIO: now reaches U1.46 (PA13)
- net SWDIO: now also J8.2 (Pin_2)
- net SWCLK: now reaches U1.49 (PA14)
- net SWCLK: now also J8.4 (Pin_4)
- net CFG21: now reaches U1.52 (PC11)
- net CFG21: now also U2.4 (CFG2)
- net CFG22: now reaches U1.8 (PC0)
- net CFG22: now also U4.4 (CFG2)
- net at C25.1, C27.1, FB2.1: now also D3.2 (A)
- new net VDC: J3.4 (Pin_4), J5.4 (Pin_4), Q1.3 (D)
- no-connect marks 6 -> 4
Other:
- note removed: "DLG-0504-101"
- moved on the sheet: D3, D4
