File: Hardware/rev2/sm4.sch (KiCad schematic (older format))
At the start: 107 parts, among them J1 Motor1, J10 CAN bus, J2 Termination, J3 CAN bus, J4 Motor1, J5 I2C, J6 Power, J7 USB_C_Receptacle_USB2.0, J8 Conn_01x05_Male, J9 I2C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

Commit message: Start improving the second rev with feedback.
Parts:
- gave numbers to parts that had none: 2
Connections:
- net MODE1 is gone; now on net VBAT: U1.17 (PA3)
- net DIR1: now also U1.20 (PA4); no longer U1.15 (PA1)
- net DIR2: now also U1.40 (PC9); no longer U1.33 (PB12)
- net VBAT: no longer U1.14 (PA0)
- net ENC2I: now reaches U1.16 (PA2)
- net ENC1A: now reaches U1.50 (PA15)
- net ENC1B: now reaches U1.55 (PB3)
- net ENC1I: now reaches U1.56 (PB4)
- net MODE2: no longer names the net of U1.43 (PA10)
- new net ENC2A: U1.14 (PA0)
- new net ENC2B: U1.15 (PA1)
- no-connect marks 44 -> 39
Changed lines of the file:
@@
 Wire Wire Line
 	15200 5800 15200 5900
-Text GLabel 2800 1300 2    50   Input ~ 0
+Text GLabel 2800 1600 2    50   Input ~ 0
 VBAT
 Text GLabel 2800 3900 2    50   Input ~ 0
@@
 Wire Wire Line
 	1300 3600 1350 3600
-Text GLabel 2800 1600 2    50   Input ~ 0
-MODE1
-Text GLabel 2800 1400 2    50   Input ~ 0
+Text GLabel 2800 1700 2    50   Input ~ 0
 DIR1
 Text GLabel 2800 4100 2    50   Input ~ 0
@@
 Wire Wire Line
 	2800 4500 2750 4500
-Text GLabel 2800 2300 2    50   Input ~ 0
-MODE2
-Text GLabel 2800 4200 2    50   Input ~ 0
+Text GLabel 1300 3900 0    50   Input ~ 0
 DIR2
 Text GLabel 2800 3700 2    50   Input ~ 0
@@
 ERR
 NoConn ~ 2750 3500
-NoConn ~ 2750 3400
-NoConn ~ 2750 3300
 NoConn ~ 2750 3200
-NoConn ~ 2750 2800
 NoConn ~ 2750 4300
 NoConn ~ 2750 4400
@@
 NoConn ~ 1350 3700
 NoConn ~ 1350 3800
-NoConn ~ 1350 3900
 NoConn ~ 1350 4000
 NoConn ~ 1350 4100
@@
 NoConn ~ 2750 3000
 Wire Wire Line
-	2800 1600 2750 1600
-Wire Wire Line
 	2800 4200 2750 4200
 $Comp
@@
 Text GLabel 2800 2200 2    50   Input ~ 0
 DRV_UART
-$Comp
-L MCU_ST_STM32F4:STM32F405RGTx U1
-U 1 1 5FF6DDC0
-P 2050 2900
-F 0 "U1" H 2600 4650 50  0000 C CNN
-F 1 "STM32F405RGTx" H 2500 1150 50  0000 C CNN
-F 2 "Package_QFP:LQFP-64_10x10mm_P0.5mm" H 1450 1200 50  0001 R CNN
-F 3 "http://www.st.com/st-web-ui/static/active/en/resource/technical/document/datasheet/DM00037051.pdf" H 2050 2900 50  0001 C CNN
-F 4 "C15742" H 2050 2900 50  0001 C CNN "LCSC"
-	1    2050 2900
-	1    0    0    -1
-$EndComp
-Wire Wire Line
-	2800 2300 2750 2300
 Text GLabel 4450 7525 0    50   Input ~ 0
 OA11
@@
 NoConn ~ 1350 3400
 NoConn ~ 1350 3500
-NoConn ~ 2750 1500
-NoConn ~ 2750 1700
-NoConn ~ 2750 1800
 NoConn ~ 2750 1900
 NoConn ~ 2750 2000
@@
 	8700 3400 8625 3400
 $Comp
-L Device:LED_Small D?
+L Device:LED_Small D1
 U 1 1 605BEF68
 P 15700 6250
-F 0 "D?" V 15746 6180 50  0000 R CNN
+F 0 "D1" V 15746 6180 50  0000 R CNN
 F 1 "LED_Small" V 15625 6250 50  0000 R CNN
 F 2 "LED_SMD:LED_0603_1608Metric_Pad1.05x0.95mm_HandSolder" V 15700 6250 50  0001 C CNN
@@
 $EndComp
 $Comp
-L Device:R_Small R?
+L Device:R_Small R9
 U 1 1 605BEF6F
 P 15700 6000
-F 0 "R?" H 15641 5954 50  0000 R CNN
+F 0 "R9" H 15641 5954 50  0000 R CNN
 F 1 "10k" H 15641 6045 50  0000 R CNN
 F 2 "Resistor_SMD:R_0402_1005Metric_Pad0.72x0.64mm_HandSolder" H 15700 6000 50  0001 C CNN
@@
 $EndComp
 $Comp
-L power:GND #PWR?
+L power:GND #PWR0132
 U 1 1 605BEF75
 P 15700 6400
-F 0 "#PWR?" H 15700 6150 50  0001 C CNN
+F 0 "#PWR0132" H 15700 6150 50  0001 C CNN
 F 1 "GND" H 15705 6227 50  0000 C CNN
 F 2 "" H 15700 6400 50  0001 C CNN
@@
 	15700 5800 15700 5900
 $Comp
-L power:VCC #PWR?
+L power:VCC #PWR0133
 U 1 1 605FA742
 P 15700 5800
-F 0 "#PWR?" H 15700 5650 50  0001 C CNN
+F 0 "#PWR0133" H 15700 5650 50  0001 C CNN
 F 1 "VCC" H 15715 5973 50  0000 C CNN
 F 2 "" H 15700 5800 50  0001 C CNN
@@
 	1    0    0    -1
 $EndComp
+NoConn ~ 2750 2300
+Text GLabel 2800 1300 2    50   Input ~ 0
+ENC2A
+Text GLabel 2800 1400 2    50   Input ~ 0
+ENC2B
+$Comp
+L MCU_ST_STM32F4:STM32F405RGTx U1
+U 1 1 5FF6DDC0
+P 2050 2900
+F 0 "U1" H 2600 4650 50  0000 C CNN
+F 1 "STM32F405RGTx" H 2500 1150 50  0000 C CNN
+F 2 "Package_QFP:LQFP-64_10x10mm_P0.5mm" H 1450 1200 50  0001 R CNN
+F 3 "http://www.st.com/st-web-ui/static/active/en/resource/technical/document/datasheet/DM00037051.pdf" H 2050 2900 50  0001 C CNN
+F 4 "C15742" H 2050 2900 50  0001 C CNN "LCSC"
+	1    2050 2900
+	1    0    0    -1
+$EndComp
+Text GLabel 2800 1500 2    50   Input ~ 0
+ENC2I
+Wire Wire Line
+	2800 1500 2750 1500
+Wire Wire Line
+	2800 1600 2750 1600
+Wire Wire Line
+	2800 1700 2750 1700
+Text GLabel 2800 2800 2    50   Input ~ 0
+ENC1A
+Text GLabel 2800 3300 2    50   Input ~ 0
+ENC1B
+Wire Wire Line
+	2800 3300 2750 3300
+Text GLabel 2800 3400 2    50   Input ~ 0
+ENC1I
+Wire Wire Line
+	2800 3400 2750 3400
+Wire Wire Line
+	1350 3900 1300 3900
+Wire Wire Line
+	2800 2800 2750 2800
+NoConn ~ 2750 1800
 $EndSCHEMATC

Commit message: Make some final touches to the rev2 hardware.
Parts:
- added J11: GPIO, Connector_PinHeader_1.27mm:PinHeader_2x05_P1.27mm_Vertical, symbol Connector_Generic:Conn_02x05_Odd_Even
- added J12: ENC_SPI, Connector_PinHeader_1.27mm:PinHeader_2x05_P1.27mm_Vertical, symbol Connector_Generic:Conn_02x05_Odd_Even
- added J13: ENC_INC, Connector_PinHeader_1.27mm:PinHeader_2x05_P1.27mm_Vertical, symbol Connector_Generic:Conn_02x05_Odd_Even
- J7: footprint Connector_USB:USB_C_Receptacle_GCT_USB4085 -> Connector_USB:USB_C_Receptacle_XKB_U262-16XN-4BVC11
- R1, R2, R3, R5: footprint Resistor_SMD:R_0603_1608Metric_Pad0.98x0.95mm_HandSolder -> Resistor_SMD:R_1206_3216Metric_Pad1.30x1.75mm_HandSolder
Connections:
- net +3V3: now also J11.4 (Pin_4), J11.6 (Pin_6), J12.10 (Pin_10), J13.1 (Pin_1), J13.2 (Pin_2)
- net +5V: now also J11.2 (Pin_2)
- net ENC1A: now also J13.3 (Pin_3)
- net ENC1B: now also J13.5 (Pin_5)
- net ENC1I: now also J13.7 (Pin_7)
- net ENC2A: now also J13.4 (Pin_4)
- net ENC2B: now also J13.6 (Pin_6)
- net ENC2I: now also J13.8 (Pin_8)
- net GND: now also J12.9 (Pin_9), J13.10 (Pin_10), J13.9 (Pin_9)
- net SCK1: now reaches U1.21 (PA5)
- net SCK1: now also J12.2 (Pin_2)
- net MISO1: now reaches U1.22 (PA6)
- net MISO1: now also J12.4 (Pin_4)
- net MOSI1: now reaches U1.23 (PA7)
- net MOSI1: now also J12.6 (Pin_6)
- net GPIO1: now reaches U1.24 (PC4)
- net GPIO1: now also J11.9 (Pin_9)
- net GPIO2: now reaches U1.25 (PC5)
- net GPIO2: now also J11.7 (Pin_7)
- net GPIO3: now reaches U1.26 (PB0)
- net GPIO3: now also J11.5 (Pin_5)
- net GPIO4: now reaches U1.27 (PB1)
- net GPIO4: now also J11.3 (Pin_3)
- net GPIO5: now reaches U1.28 (PB2)
- net GPIO5: now also J11.1 (Pin_1)
- net SCK2: now reaches U1.34 (PB13)
- net SCK2: now also J12.5 (Pin_5)
- net MISO2: now reaches U1.35 (PB14)
- net MISO2: now also J12.3 (Pin_3)
- net MOSI2: now reaches U1.36 (PB15)
- net MOSI2: now also J12.1 (Pin_1)
- net CS1: now reaches U1.38 (PC7)
- net CS1: now also J12.8 (Pin_8)
- net CS2: now reaches U1.39 (PC8)
- net CS2: now also J12.7 (Pin_7)
- new net: J11.10 (Pin_10), J11.8 (Pin_8)
- no-connect marks 39 -> 30

Commit message: Implement more of the encoder model. Make some final adjustments to rev2 board and order it.
Parts:
- D6: LCSC C72038 -> C72043
- D7: LCSC C72038 -> C2286
- R1, R2, R3, R5: LCSC C20686 -> (none)
Changed lines of the file:
@@
 F 2 "LED_SMD:LED_0603_1608Metric_Pad1.05x0.95mm_HandSolder" V 14625 6250 50  0001 C CNN
 F 3 "~" V 14625 6250 50  0001 C CNN
-F 4 "C72038" H 14625 6250 50  0001 C CNN "LCSC"
+F 4 " C72043" H 14625 6250 50  0001 C CNN "LCSC"
 	1    14625 6250
 	0    -1   -1   0
@@
 F 2 "LED_SMD:LED_0603_1608Metric_Pad1.05x0.95mm_HandSolder" V 15200 6250 50  0001 C CNN
 F 3 "~" V 15200 6250 50  0001 C CNN
-F 4 "C72038" H 15200 6250 50  0001 C CNN "LCSC"
+F 4 " C2286" H 15200 6250 50  0001 C CNN "LCSC"
 	1    15200 6250
 	0    -1   -1   0
@@
 F 2 "Resistor_SMD:R_1206_3216Metric_Pad1.30x1.75mm_HandSolder" H 5100 8250 50  0001 C CNN
 F 3 "~" H 5100 8250 50  0001 C CNN
-F 4 "C20686" H 5100 8250 50  0001 C CNN "LCSC"
+F 4 "" H 5100 8250 50  0001 C CNN "LCSC"
 	1    5100 8250
 	-1   0    0    1
@@
 F 2 "Resistor_SMD:R_1206_3216Metric_Pad1.30x1.75mm_HandSolder" H 5425 8250 50  0001 C CNN
 F 3 "~" H 5425 8250 50  0001 C CNN
-F 4 "C20686" H 5425 8250 50  0001 C CNN "LCSC"
+F 4 "" H 5425 8250 50  0001 C CNN "LCSC"
 	1    5425 8250
 	-1   0    0    1
@@
 F 2 "Resistor_SMD:R_1206_3216Metric_Pad1.30x1.75mm_HandSolder" H 10275 8275 50  0001 C CNN
 F 3 "~" H 10275 8275 50  0001 C CNN
-F 4 "C20686" H 10275 8275 50  0001 C CNN "LCSC"
+F 4 "" H 10275 8275 50  0001 C CNN "LCSC"
 	1    10275 8275
 	-1   0    0    1
@@
 F 2 "Resistor_SMD:R_1206_3216Metric_Pad1.30x1.75mm_HandSolder" H 10600 8275 50  0001 C CNN
 F 3 "~" H 10600 8275 50  0001 C CNN
-F 4 "C20686" H 10600 8275 50  0001 C CNN "LCSC"
+F 4 "" H 10600 8275 50  0001 C CNN "LCSC"
 	1    10600 8275
 	-1   0    0    1

Commit message: Write some more.
Parts:
- U6: value MCP1700-3302E_SOT23 -> MCP1700-3302
Other:
- moved on the sheet: C25, C34, C35, D3, D4, F1, FB2, Q1, U6
