File: Hardware/rev2/sm4.sch (KiCad schematic (older format))
At the start: 110 parts, among them J1 Motor1, J10 CAN bus, J11 GPIO, J12 ENC_SPI, J13 ENC_INC, J2 Termination, J3 CAN bus, J4 Motor1, J5 I2C, J6 Power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

Commit message: Finish the section on electronics design.
Parts:
- R1, R2: value 0.22 -> 0R1
Connections:
- net GND: now also J11.10 (Pin_10), J11.8 (Pin_8)
Other:
- moved on the sheet: C11, C14, C17, JP1, R4, R6, SW2, Y1
