File: Hardware/rev1/sm4.sch (KiCad schematic (older format))
At the start: 103 parts, among them J1 Motor1, J2 Termination, J3 CAN bus, J4 Motor2, J5 I2C, J6 Power, J7 USB_C_Receptacle_USB2.0, J8 Conn_01x05_Male, Q1 NDT2955, SW1 RST_SW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

Commit message: Finish the section on electronics design.
Parts:
- R3, R5: value 1R -> 0R22
Other:
- moved on the sheet: R5
Changed lines of the file:
@@
 P 3950 9100
 F 0 "R3" H 3891 9054 50  0000 R CNN
-F 1 "1R" H 3891 9145 50  0000 R CNN
+F 1 "0R22" H 3891 9145 50  0000 R CNN
 F 2 "Resistor_SMD:R_0603_1608Metric_Pad0.98x0.95mm_HandSolder" H 3950 9100 50  0001 C CNN
 F 3 "~" H 3950 9100 50  0001 C CNN
@@
 L Device:R_Small R5
 U 1 1 5FF85253
-P 4200 9100
-F 0 "R5" H 4141 9054 50  0000 R CNN
-F 1 "1R" H 4141 9145 50  0000 R CNN
-F 2 "Resistor_SMD:R_0603_1608Metric_Pad0.98x0.95mm_HandSolder" H 4200 9100 50  0001 C CNN
-F 3 "~" H 4200 9100 50  0001 C CNN
-F 4 "C20686" H 4200 9100 50  0001 C CNN "LCSC"
-	1    4200 9100
+P 4275 9100
+F 0 "R5" H 4216 9054 50  0000 R CNN
+F 1 "0R22" H 4216 9145 50  0000 R CNN
+F 2 "Resistor_SMD:R_0603_1608Metric_Pad0.98x0.95mm_HandSolder" H 4275 9100 50  0001 C CNN
+F 3 "~" H 4275 9100 50  0001 C CNN
+F 4 "C20686" H 4275 9100 50  0001 C CNN "LCSC"
+	1    4275 9100
 	-1   0    0    1
 $EndComp
@@
 L power:GND #PWR018
 U 1 1 5FF96E4A
-P 4200 9300
-F 0 "#PWR018" H 4200 9050 50  0001 C CNN
-F 1 "GND" H 4205 9127 50  0000 C CNN
-F 2 "" H 4200 9300 50  0001 C CNN
-F 3 "" H 4200 9300 50  0001 C CNN
-	1    4200 9300
-	1    0    0    -1
-$EndComp
-Wire Wire Line
-	4200 9200 4200 9300
+P 4275 9300
+F 0 "#PWR018" H 4275 9050 50  0001 C CNN
+F 1 "GND" H 4280 9127 50  0000 C CNN
+F 2 "" H 4275 9300 50  0001 C CNN
+F 3 "" H 4275 9300 50  0001 C CNN
+	1    4275 9300
+	1    0    0    -1
+$EndComp
+Wire Wire Line
+	4275 9200 4275 9300
 Wire Wire Line
 	3950 9200 3950 9300
 Wire Wire Line
-	3350 8350 4200 8350
-Wire Wire Line
 	3350 8400 3950 8400
 Wire Wire Line
 	3950 8400 3950 9000
 Wire Wire Line
-	4200 8350 4200 9000
+	4275 8350 4275 9000
 $Comp
 L power:VCC #PWR06
@@
 Text GLabel 11425 5825 0    50   Input ~ 0
 SCL
+Wire Wire Line
+	3350 8350 4275 8350
 $EndSCHEMATC
